File: hw/triangle_flywheel_balancer.kicad_sch (KiCad schematic)
At the start: 0 parts

Commit message: Project init
Parts:
- added C1, C7, C8: 1uF, triangle_flywheel_balancer:C_0603_1608Metric, symbol triangle_flywheel_balancer:C
- added C10, C11: 22uF, triangle_flywheel_balancer:C_0805_2012Metric, symbol triangle_flywheel_balancer:C
- added C12, C14, C17, C18, C19, C20, C21, C3, C6: 100nF, triangle_flywheel_balancer:C_0402_1005Metric, symbol triangle_flywheel_balancer:C
- added C13: 100uF, triangle_flywheel_balancer:C_1210_3225Metric, symbol triangle_flywheel_balancer:C
- added C15: 22nF, triangle_flywheel_balancer:C_0402_1005Metric, symbol triangle_flywheel_balancer:C
- added C16: 1nF, triangle_flywheel_balancer:C_0402_1005Metric, symbol triangle_flywheel_balancer:C
- added C2, C9: 10uF, triangle_flywheel_balancer:C_0805_2012Metric, symbol triangle_flywheel_balancer:C
- added C4, C5: 4.7uF, triangle_flywheel_balancer:C_0603_1608Metric, symbol triangle_flywheel_balancer:C
- added D1: USBLC6-2SC6, triangle_flywheel_balancer:SOT-23-6, symbol triangle_flywheel_balancer:USBLC6-2SC6
- added D2, D3: LED, triangle_flywheel_balancer:LED_0603_1608Metric, symbol triangle_flywheel_balancer:LED
- added J1: TYPE-C-31-M-12, triangle_flywheel_balancer:USB_C_Receptacle_HRO_TYPE-C-31-M-12, symbol triangle_flywheel_balancer:USB_C_Receptacle_USB2.0_16P
- added J2: BATTERY, triangle_flywheel_balancer:JST_PH_B2B-PH-K_1x02_P2.00mm_Vertical, symbol triangle_flywheel_balancer:Conn_01x02
- added J3: MOTOR, triangle_flywheel_balancer:JST_PH_B2B-PH-K_1x02_P2.00mm_Vertical, symbol triangle_flywheel_balancer:Conn_01x02
- added J4: SERVO, triangle_flywheel_balancer:PinHeader_1x03_P2.54mm_Vertical, symbol triangle_flywheel_balancer:Conn_01x03
- added J5: LATCH, triangle_flywheel_balancer:PinHeader_1x02_P2.54mm_Vertical, symbol triangle_flywheel_balancer:Conn_01x02
- added J6: OPEN, triangle_flywheel_balancer:PinHeader_1x02_P2.54mm_Vertical, symbol triangle_flywheel_balancer:Conn_01x02
- added J7: CLOSED, triangle_flywheel_balancer:PinHeader_1x02_P2.54mm_Vertical, symbol triangle_flywheel_balancer:Conn_01x02
- added L1: 1uH, triangle_flywheel_balancer:L_Murata_DFE201610P, symbol triangle_flywheel_balancer:L
- added Q1: FS8205A, triangle_flywheel_balancer:TSSOP-8_4.4x3mm_P0.65mm, symbol triangle_flywheel_balancer:FS8205A
- added R1: 10k, triangle_flywheel_balancer:R_0402_1005Metric, symbol triangle_flywheel_balancer:R
- added R10, R14, R17, R18, R19, R4, R7: 1k, triangle_flywheel_balancer:R_0402_1005Metric, symbol triangle_flywheel_balancer:R
- added R11: 33k, triangle_flywheel_balancer:R_0402_1005Metric, symbol triangle_flywheel_balancer:R
- added R12: 51k, triangle_flywheel_balancer:R_0402_1005Metric, symbol triangle_flywheel_balancer:R
- added R13, R15, R16: 100k, triangle_flywheel_balancer:R_0402_1005Metric, symbol triangle_flywheel_balancer:R
- added R2, R3: 5.1k, triangle_flywheel_balancer:R_0402_1005Metric, symbol triangle_flywheel_balancer:R
- added R5: 2k, triangle_flywheel_balancer:R_0402_1005Metric, symbol triangle_flywheel_balancer:R
- added R6: 330, triangle_flywheel_balancer:R_0402_1005Metric, symbol triangle_flywheel_balancer:R
- added R8: 1.1M, triangle_flywheel_balancer:R_0402_1005Metric, symbol triangle_flywheel_balancer:R
- added R9: 150k, triangle_flywheel_balancer:R_0402_1005Metric, symbol triangle_flywheel_balancer:R
- added S4: SW_Push, triangle_flywheel_balancer:SW_Push_1TS009xxxx-xxxx-xxxx_6x6x5mm, symbol triangle_flywheel_balancer:SW_Push
- added U1: ESP32-C3-MINI-1-N4, triangle_flywheel_balancer:ESP32-C3-MINI-1, symbol triangle_flywheel_balancer:ESP32-C3-MINI-1
- added U2: DRV8876PWPR, triangle_flywheel_balancer:HTSSOP-16-1EP_4.4x5mm_P0.65mm_EP3.4x5mm_Mask3x3mm_ThermalVias, symbol triangle_flywheel_balancer:DRV8876
- added U3: TLV7041DCKR, triangle_flywheel_balancer:SOT-353_SC-70-5, symbol triangle_flywheel_balancer:TLV7041DCK
- added U4: MCP73831T-2ACI/OT, triangle_flywheel_balancer:SOT-23-5, symbol triangle_flywheel_balancer:MCP73831-2-OT
- added U5: DW01A, triangle_flywheel_balancer:SOT-23-6, symbol triangle_flywheel_balancer:DW01A
- added U6: XC6220B331MR-G, triangle_flywheel_balancer:SOT-23-5, symbol triangle_flywheel_balancer:XC6220B331MR
- added U7: TPS61023DRLR, triangle_flywheel_balancer:SOT-563, symbol triangle_flywheel_balancer:TPS61023
Connections:
- new net: Q1.1 (D12), Q1.8 (D12)
- new net +3V3: C17.1, C2.1, C3.1, C8.1, R1.1, R11.1, R13.1, R14.1, U1.3 (3V3), U2.5 (VREF), U3.5 (V+), U6.5 (VOUT)
- new net +5V: C10.1, C11.1, C12.1, C13.1, C14.2, J4.2 (Pin_2), R8.1, U2.11 (VM), U7.6 (VOUT)
- new net BATT_N: C6.2, J2.2 (Pin_2), Q1.2 (S1), Q1.3 (S1), U5.6 (GND)
- new net BOOST_EN: U1.31 (GPIO21/U0TXD), U7.2 (EN)
- new net BOOST_FB: R8.2, R9.1, U7.1 (FB)
- new net BOOST_SW: L1.2, U7.5 (SW)
- new net BUTTON: S4.1, U1.23 (GPIO9)
- new net CC1: J1.A5 (CC1), R2.1
- new net CC2: J1.B5 (CC2), R3.1
- new net CHG_A: D2.2 (A), R4.2
- new net CPH: C15.1, U2.13 (CPH)
- new net CPL: C15.2, U2.14 (CPL)
- new net DRV_NSLEEP: U1.30 (GPIO20/U0RXD), U2.3 (nSLEEP)
- new net DW01_VDD: C6.1, R6.2, U5.5 (VCC)
- new net EN: C1.1, R1.2, U1.8 (EN/CHIP_PU)
- new net GND: C1.2, C10.2, C11.2, C12.2, C13.2, C16.2, C17.2, C18.2, C19.2, C2.2, C20.2, C21.2, C3.2, C4.2, C5.2, C7.2, C8.2, C9.2, D1.2 (GND), J1.A1 (GND), J1.A12 (GND), J1.B1 (GND), J1.B12 (GND), J1.SH (SHIELD), J4.3 (Pin_3), J5.2 (Pin_2), J6.2 (Pin_2), J7.2 (Pin_2), Q1.6 (S2), Q1.7 (S2), R10.2, R12.2, R16.2, R2.2, R3.2, R5.2, R7.2, R9.2, S4.2, U1.1 (GND), U1.11 (GND), U1.14 (GND), U1.2 (GND), U1.36 (GND), U1.37 (GND), U1.38 (GND), U1.39 (GND), U1.40 (GND), U1.41 (GND), U1.42 (GND), U1.43 (GND), U1.44 (GND), U1.45 (GND), U1.46 (GND), U1.47 (GND), U1.48 (GND), U1.49 (GND), U1.50 (GND), U1.51 (GND), U1.52 (GND), U1.53 (GND), U2.15 (GND), U2.16 (PMODE), U2.17 (PAD), U2.7 (IMODE), U2.9 (PGND), U3.2 (V-), U4.2 (V_{SS}), U6.2 (GND), U7.4 (GND)
- new net IPROPI: C16.1, R10.1, U1.13 (GPIO1/ADC1_CH1/XTAL_32K_N), U2.6 (IPROPI), U3.3 (+)
- new net LED_A: D3.2 (A), R14.2
- new net MOTOR_A: J3.1 (Pin_1), U2.8 (OUT1)
- new net MOTOR_B: J3.2 (Pin_2), U2.10 (OUT2)
- new net MOTOR_EN: U1.20 (GPIO6), U2.1 (EN/IN1)
- new net MOTOR_PH: U1.21 (GPIO7), U2.2 (PH/IN2)
- new net PROG: R5.1, U4.5 (PROG)
- new net PROT_CS: R7.1, U5.2 (CS)
- new net PROT_OC: Q1.5 (G2), U5.3 (OC)
- new net PROT_OD: Q1.4 (G1), U5.1 (OD)
- new net SERVO_PWM: J4.1 (Pin_1), U1.16 (GPIO10)
- new net STAT: D2.1 (K), U4.1 (STAT)
- new net STATUS_LED: D3.1 (K), U1.22 (GPIO8)
- new net SW_CLOSED: C21.1, R19.2, U1.19 (GPIO5/ADC2_CH0)
- new net SW_CLOSED_J: J7.1 (Pin_1), R19.1
- new net SW_LATCH: C19.1, R17.2, U1.6 (GPIO3/ADC1_CH3)
- new net SW_LATCH_J: J5.1 (Pin_1), R17.1
- new net SW_OPEN: C20.1, R18.2, U1.18 (GPIO4/ADC1_CH4)
- new net SW_OPEN_J: J6.1 (Pin_1), R18.1
- new net USB_DM: D1.6 (I/O1), U1.26 (GPIO18/USB_D-)
- new net USB_DM_C: D1.1 (I/O1), J1.A7 (D-), J1.B7 (D-)
- new net USB_DP: D1.4 (I/O2), U1.27 (GPIO19/USB_D+)
- new net USB_DP_C: D1.3 (I/O2), J1.A6 (D+), J1.B6 (D+)
- new net VBAT: C5.1, C7.1, C9.1, J2.1 (Pin_1), L1.1, R15.1, R6.1, U4.3 (V_{BAT}), U6.1 (VIN), U6.3 (CE), U7.3 (VIN)
- new net VBAT_SENSE: C18.1, R15.2, R16.1, U1.12 (GPIO0/ADC1_CH0/XTAL_32K_P)
- new net VBUS: C4.1, D1.5 (VBUS), J1.A4 (VBUS), J1.A9 (VBUS), J1.B4 (VBUS), J1.B9 (VBUS), R4.1, U4.4 (V_{DD})
- new net VCP: C14.1, U2.12 (VCP)
- new net VTH: R11.2, R12.1, U3.4 (-)
- new net nFAULT_ANY: R13.2, U1.5 (GPIO2/ADC1_CH2), U2.4 (nFAULT), U3.1
- no-connect marks 0 -> 18

Commit message: Upd
Parts:
- added C22: 100nF, triangle_flywheel_balancer:C_0402_1005Metric, symbol triangle_flywheel_balancer:C
- added R20: 68k, triangle_flywheel_balancer:R_0402_1005Metric, symbol triangle_flywheel_balancer:R
- added R21: 100k, triangle_flywheel_balancer:R_0402_1005Metric, symbol triangle_flywheel_balancer:R
- C1, C7, C8: LCSC Part C5673 -> C15849; MPN CL10A105KA8NNNC -> CL10A105KB8NNNC
- R8: value 1.1M -> 110k; LCSC Part (none) -> C25745; MPN RC0402FR-071M1L -> 0402WGF1103TCE; Manufacturer YAGEO -> UNI-ROYAL
- R9: value 150k -> 15k; LCSC Part C93947 -> C25756; MPN RC0402FR-07150KL -> 0402WGF1502TCE; Manufacturer YAGEO -> UNI-ROYAL
- U3: value TLV7041DCKR -> TLV1701AIDBVR; footprint triangle_flywheel_balancer:SOT-353_SC-70-5 -> triangle_flywheel_balancer:SOT-23-5; symbol triangle_flywheel_balancer:TLV7041DCK -> triangle_flywheel_balancer:TLV1701; LCSC Part (none) -> C130035; MPN TLV7041DCKR -> TLV1701AIDBVR
Connections:
- net +3V3: now also U2.3 (nSLEEP)
- net GND: now also C22.2, R21.2
- net IPROPI: now also U3.1 (+); no longer U3.3 (+)
- net VBUS: now also R20.1
- net VTH: now also U3.3 (-); no longer U3.4 (-)
- net nFAULT_ANY: now also U3.4; no longer U3.1
- net DRV_NSLEEP renamed VBUS_DET
- net VBUS_DET: now also C22.1, R20.2, R21.1; no longer U2.3 (nSLEEP)
